Commit message: Модель погрузчика с цилиндрическим корпусом и возможностью управлять поворотом колеса и скоростью. Самонаправляющиеся колеса

File: description/pallet.urdf.xacro (robot description, xacro)
@@ -1,5 +1,5 @@
 <?xml version="1.0"?>
-<robot xmlns:xacro="http://www.ros.org/wiki/xacro" name="mecanum">
+<robot xmlns:xacro="http://www.ros.org/wiki/xacro" name="pallet">
     <xacro:include filename="pallet_core.xacro"/>
-<!--    <xacro:include filename="ros2_control.xacro"/>-->
+    <xacro:include filename="ros2_control.xacro"/>
  </robot>

File: description/pallet_core.xacro (robot description, xacro)
@@ -1,10 +1,13 @@
 <?xml version="1.0"?>
-<robot xmlns:xacro="http://www.ros.org/wiki/xacro" name="mecanum">
+<robot xmlns:xacro="http://www.ros.org/wiki/xacro" name="pallet">
+<!--    Макрос для расчета инерции простых фигур-->
+    <xacro:include filename="inertial_macros.xacro"/>
     <material name="gray">
-        <color rgba="66 60 63 0.8"/>
+        <color rgba="0.66 0.60 0.63 1"/>
     </material>
     <material name="black">
-        <color rgba="41 41 41 0.97"/>
+        <color rgba="0.41 0.41 0.41 1"/>
     </material>
+    <!-- BASE LINK -->
     <link name="base_link">
     </link>
@@ -14,12 +17,193 @@
         <origin xyz="0 0 0"/>
     </joint>
+                  <!-- Корпус робота -->
     <link name="body_link">
         <visual>
-            <origin xyz="0 0 0"/>
-            <geometry>
-                <cylinder radius="0.6" length="1"/>
+            <origin xyz="0.2 -0.3 0" rpy=" 0 0 ${pi/2} "/>
+            <geometry>
+                 <mesh filename="file://$(find sm_robotics)/description/meshes/body.stl" scale="0.01 0.01 0.01" />
+<!--                <cylinder radius="0.6" length="1"/>-->
             </geometry>
             <material name="gray"/>
         </visual>
-    </link>
+        <collision>
+            <origin xyz="0 0 0.5" rpy=" 0 0 0 "/>
+            <geometry>
+                 <box size="0.35 0.56 1"/>
+            </geometry>
+        </collision>
+        <xacro:inertial_box mass="100" x="0.35" y="0.56" z="1">
+            <origin xyz="0.2 -0.3 0" rpy="0 0 ${pi/2}"/>
+        </xacro:inertial_box>
+    </link>
+    <gazebo reference="body_link">
+        <material>Gazebo/Red</material>
+        <mu1 value="0.001"/>
+        <mu2 value="0.001"/>
+    </gazebo>
+    <!-- WHEELS LINK -->
+                <!--Привод поворота-->
+    <joint name="steering_joint" type="continuous">
+        <parent link="base_link"/>
+        <child link="steering_link"/>
+        <origin xyz="0.05 0 0.1" rpy="0 0 0"/>
+        <axis xyz="0 0 1"/>
+    </joint>
+    <link name="steering_link">
+<!--        пустой объект, без которого не работает модель в газебо-->
+        <visual>
+            <origin xyz="0 0 0.15" rpy=" 0 0 0 "/>
+            <geometry>
+                <cylinder radius="0.1" length="0.03"/>
+            </geometry>
+            <material name="black"/>
+        </visual>
+        <collision>
+            <origin xyz="0 0 0" rpy=" 0 0 0 "/>
+            <geometry>
+                <cylinder radius="0.01" length="0.01"/>
+            </geometry>
+        </collision>
+        <xacro:inertial_cylinder mass="5" length="0.1" radius="0.1">
+            <origin xyz="0 0 0" rpy="0 0 0"/>
+        </xacro:inertial_cylinder>
+    </link>
+            <!--    Мотор-колесо-->
+    <joint name="drive_wheel_joint" type="continuous">
+        <parent link="steering_link"/>
+<!--        <parent link="base_link"/>-->
+        <child link="drive_wheel_link"/>
+<!--         <origin xyz="0.05 0 0.1" rpy="-${pi/2} 0 0"/>-->
+        <origin xyz="0 0 0" rpy="-${pi/2} 0 0"/>
+        <axis xyz="0 0 1"/>
+    </joint>
+    <link name="drive_wheel_link">
+        <visual>
+            <origin xyz="0 0 0" rpy=" 0 0 0 "/>
+            <geometry>
+                <cylinder radius="0.1" length="0.1"/>
+            </geometry>
+            <material name="black"/>
+        </visual>
+        <collision>
+            <origin xyz="0 0 0" rpy=" 0 0 0 "/>
+            <geometry>
+                <cylinder radius="0.1" length="0.1"/>
+            </geometry>
+        </collision>
+        <xacro:inertial_cylinder mass="5" length="0.1" radius="0.1">
+            <origin xyz="0 0 0" rpy="0 0 0"/>
+        </xacro:inertial_cylinder>
+    </link>
+    <gazebo reference="drive_wheel_link">
+        <material>Gazebo/Orange</material>
+    </gazebo>
+             <!-- Самонаправляющиеся колеса -->
+    <joint name="right_caster_joint" type="fixed">
+        <parent link="base_link"/>
+        <child link="right_caster_link"/>
+        <origin xyz="-0.1 -0.1 0.04"/>
+    </joint>
+    <link name="right_caster_link">
+        <visual>
+            <origin xyz="0 0 0" rpy=" 0 0 0 "/>
+            <geometry>
+                <sphere radius="0.04"/>
+            </geometry>
+            <material name="black"/>
+        </visual>
+        <collision>
+            <origin xyz="0 0 0" rpy=" 0 0 0 "/>
+            <geometry>
+                <sphere radius="0.04"/>
+            </geometry>
+        </collision>
+        <xacro:inertial_sphere mass="1"  radius="0.04">
+            <origin xyz="0 0 0" rpy="0 0 0"/>
+        </xacro:inertial_sphere>
+    </link>
+    <gazebo reference="right_caster_link">
+        <material>Gazebo/Black</material>
+        <mu1 value="0.001"/>
+        <mu2 value="0.001"/>
+    </gazebo>
+    <joint name="left_caster_joint" type="fixed">
+        <parent link="base_link"/>
+        <child link="left_caster_link"/>
+        <origin xyz="-0.1 0.1 0.04"/>
+    </joint>
+    <link name="left_caster_link">
+        <visual>
+            <origin xyz="0 0 0" rpy=" 0 0 0 "/>
+            <geometry>
+                <sphere radius="0.04"/>
+            </geometry>
+            <material name="black"/>
+        </visual>
+        <collision>
+            <origin xyz="0 0 0" rpy=" 0 0 0 "/>
+            <geometry>
+                <sphere radius="0.04"/>
+            </geometry>
+        </collision>
+        <xacro:inertial_sphere mass="1"  radius="0.04">
+            <origin xyz="0 0 0" rpy="0 0 0"/>
+        </xacro:inertial_sphere>
+    </link>
+    <gazebo reference="left_caster_link">
+        <material>Gazebo/Black</material>
+        <mu1 value="0.001"/>
+        <mu2 value="0.001"/>
+    </gazebo>
+                <!--  Вилы -->
+    <joint name="right_fork_joint" type="prismatic">
+        <parent link="base_link"/>
+        <child link="right_fork_link"/>
+        <origin xyz="-0.45 -0.14 0.03" rpy="0 0 0"/>
+        <axis xyz="0 0 1"/>
+        <limit lower="0" upper="0.5" velocity="100" effort="100"/>
+    </joint>
+        <link name="right_fork_link">
+        <visual>
+            <geometry>
+                <box size="0.6 0.08 0.03" />
+            </geometry>
+            <material name="black"/>
+        </visual>
+        <collision>
+            <origin xyz="0 0 0" rpy=" 0 0 0 "/>
+            <geometry>
+                 <box size="0.6 0.08 0.03"/>
+            </geometry>
+        </collision>
+        <xacro:inertial_box mass="4" x="0.6" y="0.08" z="0.03">
+            <origin xyz="0 0 0" rpy="0 0 0"/>
+        </xacro:inertial_box>
+    </link>
+    <joint name="left_fork_joint" type="fixed">
+        <parent link="right_fork_link"/>
+        <child link="left_fork_link"/>
+        <origin xyz="0 0.28 0"/>
+    </joint>
+        <link name="left_fork_link">
+        <visual>
+            <geometry>
+                <box size="0.6 0.08 0.03" />
+            </geometry>
+            <material name="black"/>
+        </visual>
+        <collision>
+            <origin xyz="0 0 0" rpy=" 0 0 0 "/>
+            <geometry>
+                 <box size="0.6 0.08 0.03"/>
+            </geometry>
+        </collision>
+        <xacro:inertial_box mass="4" x="0.6" y="0.08" z="0.03">
+            <origin xyz="0 0 0" rpy="0 0 0"/>
+        </xacro:inertial_box>
+    </link>
+<!--    "Покраска модели в Gazebo"-->
+<!--    <gazebo refrence="left_fork_link">-->
+<!--        <material>Gazebo/Blue</material>-->
+<!--    </gazebo>-->
  </robot>
